File: LED-Polyhedron.kicad_pcb (KiCad board)
At the start: 2 copper layers, 91.7 x 92.3 mm, 44 parts, among them J1 IN, J2 IN, U1 TPS-DC-DC

Commit message: added topor files
Parts:
- removed ?: , otter:polyhedrone
- added C23: C, Capacitor_SMD:C_0603_1608Metric, F.Cu at (56.1, 75.8)
- added D19: WS2812B, LED_SMD:LED_WS2812B_PLCC4_5.0x5.0mm_P3.2mm, F.Cu at (54.7, 79.8)
- added otter: otter, , F.Cu at (0.00, 0.00)
- moved C20 12.5 mm to (74.0, 62.9), turned to 315 degrees
- moved C7 8.34 mm to (32.8, 38.0)
- moved D16 4.14 mm to (72.4, 66.7), turned to 315 degrees
Connections:
- D15 pad 2: /sheet5DBB0857/DIN -> /sheet5DD4437B/DIN
Routing:
- net GND: track 0.00 -> 543.3 mm, vias 0 -> 31
- net VCC: track 8.11 -> 347.3 mm, vias 0 -> 14
- net /sheet5DBA4166/DIN: track 0.00 -> 27.8 mm
- net /sheet5DB72310/DIN: track 0.00 -> 19.0 mm
- net /sheet5DB71B84/DIN: track 0.00 -> 18.8 mm
- net /sheet5DBB0857/DIN: track 0.00 -> 18.6 mm
- net /sheet5DB7230F/DIN: track 0.00 -> 18.2 mm
- net /sheet5DBB211F/DIN: track 0.00 -> 18.0 mm
- net /sheet5DD4437B/DIN: track 0.00 -> 17.0 mm
- net /sheet5DB71B86/DIN: track 0.00 -> 14.9 mm
- net /sheet5DB71B88/DIN: track 0.00 -> 14.1 mm
- net /sheet5DB71B85/DIN: track 0.00 -> 14.0 mm
- net /sheet5DB72312/DIN: track 0.00 -> 13.3 mm
- net /sheet5DB71767/DIN: track 0.00 -> 13.2 mm
- net /sheet5DB718FF/DIN: track 0.00 -> 12.9 mm
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- added copper zone on B.Cu, net GND
- added copper zone on F.Cu, net GND
